File: Analogue-Inputs.kicad_sch (KiCad schematic)
At the start: 58 parts, among them J601 1-1337535-0, J602 1-1337535-0, J603 1-1337535-0, U601 TSV912AIDR, U602 TSV912AIDR, U603 LM358LVIDR, U604 TSV912AIDR, U605 TSV912AIDR

Commit message: feat: checked REV A
Changed lines of the file:
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@@
+		)
+	)
+	(text_box "DESIGN NOTE:\nThe 0.61V VREF is generated to bias the output to 0.61V, with A_{v} ≈ 24.9 this gives a maximal headroom."
+		(exclude_from_sim no)
+		(at 250.19 113.03 0)
+		(size 63.5 8.89)
+		(margins 1.3525 1.3525 1.3525 1.3525)
+		(stroke
+			(width 0.8)
+			(type solid)
+			(color 200 200 200 1)
+		)
+		(fill
+			(type none)
+		)
+		(effects
+			(font
+				(face "Arial")
+				(size 1.27 1.27)
+				(color 0 0 0 1)
+			)
+			(justify left top)
 		)
 	)
