File: Analogue-Outputs.kicad_sch (KiCad schematic)
At the start: 18 parts, among them J701 PH1-02-UA, U701 LM358LVIDR, U702 LM358LVIDR

Commit message: feat: checked REV A
Parts:
- added R709: 100, Resistor_SMD:R_0603_1608Metric, symbol Device:R
- renumbered C708 to C707
Connections:
- net SHAKER_N: now also R709.2
- net SHAKER_P: now also R709.1
Other:
- moved on the sheet: J701
Changed lines of the file:
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@@
 	)
 	(rectangle
+		(start 229.87 78.74)
+		(end 242.57 96.52)
+		(stroke
+			(width 0)
+			(type dash)
+			(color 255 0 0 1)
+		)
+		(fill
+			(type none)
+		)
+	)
+	(rectangle
 		(start 58.42 35.56)
 		(end 167.64 86.36)
@@
 	(rectangle
 		(start 168.91 58.42)
-		(end 238.76 124.46)
+		(end 269.24 124.46)
 		(stroke
 			(width 0)
@@
 		)
 	)
+	(text_box "DESIGN NOTE:\nOptional 100R load direct on board."
+		(exclude_from_sim no)
+		(at 246.38 102.87 0)
+		(size 21.59 10.16)
+		(margins 2 2 2 2)
+		(stroke
+			(width 1)
+			(type solid)
+			(color 255 165 0 1)
+		)
+		(fill
+			(type none)
+		)
+		(effects
+			(font
+				(face "Arial")
+				(size 1.27 1.27)
+				(color 0 0 0 1)
+			)
+			(justify left top)
+		)
+	)
 	(text_box "[${#}] ${TITLE}"
 		(exclude_from_sim no)
@@
 	(text_box "DESIGN NOTE:\nLM358LVIDR can supply up to 40mA, for the differential driver this should be enough to provide 4 Vpp to the 100R shaker load."
 		(exclude_from_sim no)
-		(at 240.03 58.42 0)
+		(at 238.76 59.69 0)
 		(size 29.21 12.7)
 		(margins 1.3525 1.3525 1.3525 1.3525)
@@
 	)
 	(junction
+		(at 238.76 74.93)
+		(diameter 0)
+		(color 0 0 0 0)
+	)
+	(junction
 		(at 166.37 72.39)
 		(diameter 0)
@@
 	)
 	(junction
+		(at 238.76 100.33)
+		(diameter 0)
+		(color 0 0 0 0)
+	)
+	(junction
 		(at 203.2 113.03)
 		(diameter 0)
@@
 	(wire
 		(pts
-			(xy 234.95 88.9) (xy 242.57 88.9)
+			(xy 228.6 100.33) (xy 238.76 100.33)
 		)
 		(stroke
@@
 	(wire
 		(pts
+			(xy 247.65 88.9) (xy 247.65 100.33)
+		)
+		(stroke
+			(width 0)
+			(type default)
+		)
+	)
+	(wire
+		(pts
 			(xy 85.09 121.92) (xy 85.09 114.3)
 		)
@@
 		)
 	)
+	(polyline
+		(pts
+			(xy 246.38 102.87) (xy 242.57 96.52)
+		)
+		(stroke
+			(width 0)
+			(type dash)
+			(color 255 0 0 1)
+		)
+	)
 	(wire
 		(pts
@@
 	(wire
 		(pts
-			(xy 234.95 74.93) (xy 234.95 86.36)
+			(xy 247.65 88.9) (xy 250.19 88.9)
 		)
 		(stroke
@@
 	(wire
 		(pts
-			(xy 228.6 100.33) (xy 234.95 100.33)
+			(xy 184.15 97.79) (xy 184.15 100.33)
 		)
 		(stroke
@@
 	(wire
 		(pts
-			(xy 184.15 97.79) (xy 184.15 100.33)
+			(xy 223.52 100.33) (xy 228.6 100.33)
 		)
 		(stroke
@@
 	(wire
 		(pts
-			(xy 234.95 100.33) (xy 234.95 88.9)
+			(xy 238.76 100.33) (xy 238.76 91.44)
 		)
 		(stroke
@@
 	(wire
 		(pts
-			(xy 57.15 67.31) (xy 59.69 67.31)
+			(xy 228.6 74.93) (xy 238.76 74.93)
 		)
 		(stroke
@@
 	(wire
 		(pts
-			(xy 208.28 102.87) (xy 203.2 102.87)
+			(xy 57.15 67.31) (xy 59.69 67.31)
 		)
 		(stroke
@@
 	(wire
 		(pts
-			(xy 208.28 77.47) (xy 203.2 77.47)
+			(xy 208.28 102.87) (xy 203.2 102.87)
 		)
 		(stroke
@@
 	(wire
 		(pts
-			(xy 228.6 74.93) (xy 234.95 74.93)
+			(xy 208.28 77.47) (xy 203.2 77.47)
 		)
 		(stroke
@@
 	(wire
 		(pts
-			(xy 228.6 74.93) (xy 223.52 74.93)
+			(xy 184.15 97.79) (xy 208.28 97.79)
 		)
 		(stroke
@@
 	(wire
 		(pts
-			(xy 184.15 97.79) (xy 208.28 97.79)
+			(xy 147.32 74.93) (xy 148.59 74.93)
 		)
 		(stroke
@@
 	(wire
 		(pts
-			(xy 147.32 74.93) (xy 148.59 74.93)
+			(xy 86.36 67.31) (xy 86.36 69.85)
 		)
 		(stroke
@@
 	(wire
 		(pts
-			(xy 86.36 67.31) (xy 86.36 69.85)
+			(xy 46.99 101.6) (xy 46.99 102.87)
 		)
 		(stroke
@@
 	(wire
 		(pts
-			(xy 234.95 86.36) (xy 242.57 86.36)
+			(xy 238.76 100.33) (xy 247.65 100.33)
 		)
 		(stroke
@@
 	(wire
 		(pts
-			(xy 46.99 101.6) (xy 46.99 102.87)
+			(xy 72.39 119.38) (xy 72.39 121.92)
 		)
 		(stroke
@@
 	(wire
 		(pts
-			(xy 72.39 119.38) (xy 72.39 121.92)
+			(xy 247.65 74.93) (xy 247.65 86.36)
+		)
+		(stroke
+			(width 0)
+			(type default)
+		)
+	)
+	(wire
+		(pts
+			(xy 223.52 74.93) (xy 228.6 74.93)
 		)
 		(stroke
@@
 	(wire
 		(pts
+			(xy 247.65 86.36) (xy 250.19 86.36)
+		)
+		(stroke
+			(width 0)
+			(type default)
+		)
+	)
+	(wire
+		(pts
 			(xy 59.69 102.87) (xy 59.69 106.68)
 		)
@@
 	(wire
 		(pts
-			(xy 223.52 100.33) (xy 228.6 100.33)
+			(xy 238.76 74.93) (xy 238.76 83.82)
 		)
 		(stroke
@@
 	(wire
 		(pts
+			(xy 238.76 74.93) (xy 247.65 74.93)
+		)
+		(stroke
+			(width 0)
+			(type default)
+		)
+	)
+	(wire
+		(pts
 			(xy 109.22 69.85) (xy 111.76 69.85)
 		)
@@
 	)
 	(symbol
+		(lib_id "Device:R")
+		(at 238.76 87.63 0)
+		(unit 1)
+		(exclude_from_sim no)
+		(in_bom yes)
+		(on_board yes)
+		(dnp yes)
+		(property "Reference" "R709"
+			(at 236.22 85.0899 0)
+			(effects
+				(font
+					(size 1.27 1.27)
+				)
+				(justify right)
+			)
+		)
+		(property "Value" "100"
+			(at 236.22 87.6299 0)
+			(effects
+				(font
+					(size 1.27 1.27)
+				)
+				(justify right)
+			)
+		)
+		(property "Footprint" "Resistor_SMD:R_0603_1608Metric"
+			(at 236.982 87.63 90)
+			(effects
+				(font
+					(size 1.27 1.27)
+				)
+				(hide yes)
+			)
+		)
+		(property "Datasheet" "https://www.analogtechnologies.com/document/New_Resistor_Kits.pdf"
+			(at 238.76 87.63 0)
+			(effects
+				(font
+					(size 1.27 1.27)
+				)
+				(hide yes)
+			)
+		)
+		(property "Description" "RES 100 OHM 1% 1/10W 0603"
+			(at 238.76 87.63 0)
+			(effects
+				(font
+					(size 1.27 1.27)
+				)
+				(hide yes)
+			)
+		)
+		(property "Manufacturer" "Analog Technologies"
+			(at 238.76 87.63 90)
+			(effects
+				(font
+					(size 1.27 1.27)
+				)
+				(hide yes)
+			)
+		)
+		(property "Tolerance" "1%"
+			(at 236.22 90.1699 0)
+			(effects
+				(font
+					(size 1.27 1.27)
+				)
+				(justify right)
+			)
+		)
+		(property "Power" "1/10W"
+			(at 238.76 87.63 90)
+			(effects
+				(font
+					(size 1.27 1.27)
+				)
+				(hide yes)
+			)
+		)
+		(pin "2"
+		)
+		(pin "1"
+		)
+		(instances
+			(project "DREAM"
+				(path "/f9e05184-c88b-4a88-ae9c-ab2bdb32be7c/c5103ceb-5325-4a84-a025-9638a412984e/8fe0aa77-1043-4de2-87da-8c916c2e1a1d"
+					(reference "R709")
+					(unit 1)
+				)
+			)
+		)
+	)
+	(symbol
 		(lib_id "power:GND")
 		(at 140.97 81.28 0)
@@
 		(on_board yes)
 		(dnp no)
-		(property "Reference" "C708"
+		(property "Reference" "C707"
 			(at 187.96 101.5999 0)
 			(effects
@@
 			(project "DREAM"
 				(path "/f9e05184-c88b-4a88-ae9c-ab2bdb32be7c/c5103ceb-5325-4a84-a025-9638a412984e/8fe0aa77-1043-4de2-87da-8c916c2e1a1d"
-					(reference "C708")
+					(reference "C707")
 					(unit 1)
 				)
@@
 	(symbol
 		(lib_id "Connector:Conn_01x02_Pin")
-		(at 247.65 86.36 0)
+		(at 255.27 86.36 0)
 		(mirror y)
 		(unit 1)
@@
 		(dnp no)
 		(property "Reference" "J701"
-			(at 248.92 88.9001 0)
+			(at 256.54 88.9001 0)
 			(effects
 				(font
@@
 		)
 		(property "Value" "PH1-02-UA"
-			(at 248.92 86.3601 0)
+			(at 256.54 86.3601 0)
 			(effects
 				(font
@@
 		)
 		(property "Footprint" "Connector_PinHeader_2.54mm:PinHeader_1x02_P2.54mm_Vertical"
-			(at 247.65 86.36 0)
+			(at 255.27 86.36 0)
 			(effects
 				(font
@@
 		)
 		(property "Datasheet" "~"
-			(at 247.65 86.36 0)
+			(at 255.27 86.36 0)
 			(effects
 				(font
@@
 			)
 		)
-		(property "Description" "Generic connector, single row, 01x02, script generated"
-			(at 247.65 86.36 0)
+		(property "Description" "HEADER 2PIN 2.54MM THT"
+			(at 255.27 86.36 0)
 			(effects
 				(font
@@
 		)
 		(property "Manufacturer" "Adam Tech"
-			(at 247.65 86.36 0)
+			(at 255.27 86.36 0)
 			(effects
 				(font
@@
 		)
 		(property "MPN" ""
-			(at 247.65 86.36 0)
+			(at 255.27 86.36 0)
 			(effects
 				(font
@@
 		(dnp no)
 		(fields_autoplaced yes)
-		(property "Reference" "#PWR0722"
+		(property "Reference" "#PWR0711"
 			(at 184.15 116.84 0)
 			(effects
@@
 			(project "DREAM"
 				(path "/f9e05184-c88b-4a88-ae9c-ab2bdb32be7c/c5103ceb-5325-4a84-a025-9638a412984e/8fe0aa77-1043-4de2-87da-8c916c2e1a1d"
-					(reference "#PWR0722")
+					(reference "#PWR0711")
 					(unit 1)
 				)
