File: Project Architecture.kicad_sch (KiCad schematic)
At the start: 0 parts

Commit message: feat: checked REV A
Other:
- title: PROJECT ARCHITECTURE -> ARCHITECTURE
Changed lines of the file:
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@@
 	(paper "A4")
 	(title_block
-		(title "PROJECT ARCHITECTURE")
+		(title "ARCHITECTURE")
 		(date "2026-04-06")
 		(rev "${REVISION}")

Commit message: fix: circuit schem as one sheet
Parts:
- added C401, C403, C501, C506, C507, C508, C509, C512, C601, C602, C604, C610, C613, C614, C616, C701, C702, C707: 100n, Capacitor_SMD:C_0603_1608Metric, symbol Device:C
- added C402, C505, C611, C612: 10u, Capacitor_SMD:C_0603_1608Metric, symbol Device:C
- added C404, C405, C511, C603, C615: 1u, Capacitor_SMD:C_0603_1608Metric, symbol Device:C
- added C502, C503: 27p, Capacitor_SMD:C_0603_1608Metric, symbol Device:C
- added C504: 4.7u, Capacitor_SMD:C_0603_1608Metric, symbol Device:C
- added C510, C705: 10n, Capacitor_SMD:C_0603_1608Metric, symbol Device:C
- added C605, C607, C608, C609: 390n, Capacitor_SMD:C_0603_1608Metric, symbol Device:C
- added C606: 180n, Capacitor_SMD:C_0603_1608Metric, symbol Device:C
- added C703: 15n, Capacitor_SMD:C_0603_1608Metric, symbol Device:C
- added C704: 18n, Capacitor_SMD:C_0603_1608Metric, symbol Device:C
- added C706: 68n, Capacitor_SMD:C_0603_1608Metric, symbol Device:C
- added D401: D3Z10BF-7, Diode_SMD:D_SOD-323_HandSoldering, symbol Device:D_Zener
- added D501, D502: LED, LED_SMD:LED_0805_2012Metric, symbol Device:LED
- added D503: TVS, Diode_SMD:D_SMB, symbol Diode:SM6T6V8A
- added D601, D602, D603, D604, D605, D606: 1N4148WS, Diode_SMD:D_SOD-323_HandSoldering, symbol Diode:1N4148WS
- added F401, F501: MF-MSMF030-2, Resistor_SMD:R_1812_4532Metric, symbol Device:Polyfuse_Small
- added FB501: BLM18KG101JH1D, Inductor_SMD:L_0603_1608Metric, symbol Device:FerriteBead_Small
- added FID401, FID402, FID403: FIDUCIAL, Fiducial:Fiducial_1mm_Mask2mm, symbol Mechanical:Fiducial
- added H401, H402, H403, H404: MOUNT_M2.5, MountingHole:MountingHole_2.7mm_M2.5_ISO7380_Pad, symbol Mechanical:MountingHole_Pad
- added ID401: BOARD_STACKUP_MARKER, RD-Symbols-Silkscreen:STACKUP_ID_2L, symbol Ryan-Dynamics:BOARD_STACKUP_MARKER
- added J401: KLDX-0202-B, Connector_BarrelJack:BarrelJack_Kycon_KLDX-0202-xC_Horizontal, symbol Connector:Barrel_Jack_Switch
- added J402: EBWA-02-B, TerminalBlock_Phoenix:TerminalBlock_Phoenix_MKDS-1-2-3.81_1x02_P3.81mm_Horizontal, symbol Connector:Screw_Terminal_01x02
- added J501: 20021121-00014T1LF, Connector_PinHeader_1.27mm:PinHeader_2x07_P1.27mm_Vertical_SMD, symbol Connector:Conn_ST_STDC14
- added J502: USB4105-GF-A, Connector_USB:USB_C_Receptacle_GCT_USB4105-xx-A_16P_TopMnt_Horizontal, symbol Connector:USB_C_Receptacle_USB2.0_16P
- added J601, J602, J603: 1-1337535-0, Connector_Coaxial:BNC_TEConnectivity_1478204_Vertical, symbol Connector:Conn_Coaxial
- added J701: PH1-02-UA, Connector_PinHeader_2.54mm:PinHeader_1x02_P2.54mm_Vertical, symbol Connector:Conn_01x02_Pin
- added JP401: PR20203BNN, Connector_PinHeader_2.54mm:PinHeader_1x03_P2.54mm_Vertical, symbol Jumper:Jumper_3_Bridged12
- added Q401: MCU18P10Y-TP, MCU18P10Y-TP:DPAK_MCC, symbol MCU18P10Y-TP:MCU18P10Y-TP
- added R401, R402, R618: 100k, Resistor_SMD:R_0603_1608Metric, symbol Device:R
- added R501, R502, R601, R602, R603, R604: 1k, Resistor_SMD:R_0603_1608Metric, symbol Device:R
- added R503, R504, R505, R506: 22.1, Resistor_SMD:R_0603_1608Metric, symbol Device:R
- added R507: 0, Resistor_SMD:R_0603_1608Metric, symbol Device:R
- added R508, R611, R613, R614, R624, R706, R707, R708: 10k, Resistor_SMD:R_0603_1608Metric, symbol Device:R
- added R509, R510, R605, R608: 5.11k, Resistor_SMD:R_0603_1608Metric, symbol Device:R
- added R606, R609: 27.4k, Resistor_SMD:R_0603_1608Metric, symbol Device:R
- added R607: 11k, Resistor_SMD:R_0603_1608Metric, symbol Device:R
- added R610, R617, R705: 20k, Resistor_SMD:R_0603_1608Metric, symbol Device:R
- added R612: 5.62k, Resistor_SMD:R_0603_1608Metric, symbol Device:R
- added R615, R619, R620, R709: 100, Resistor_SMD:R_0603_1608Metric, symbol Device:R
- added R616: 18.2k, Resistor_SMD:R_0603_1608Metric, symbol Device:R
- added R621, R622: 2.2M, Resistor_SMD:R_0603_1608Metric, symbol Device:R
- added R623: 39.2k, Resistor_SMD:R_0603_1608Metric, symbol Device:R
- added R701, R702: 12.1k, Resistor_SMD:R_0603_1608Metric, symbol Device:R
- added R703, R704: 7.5k, Resistor_SMD:R_0603_1608Metric, symbol Device:R
- added SW501: PTS526SK15SMTR2 LFS, PTS526SxxxSMTR2:SW_SPST_PTS526xxxSMTR, symbol Switch:SW_Push
- added TP401: VBATT_RAW, RD-Testpoints:TestPoint_Pad_D1.0mm, symbol Connector:TestPoint
- added TP402: VBATT, RD-Testpoints:TestPoint_Pad_D1.0mm, symbol Connector:TestPoint
- added TP403: +3V0, RD-Testpoints:TestPoint_Pad_D1.0mm, symbol Connector:TestPoint
- added TP404: GND, RD-Testpoints:TestPoint_Pad_1.0x1.0mm, symbol Connector:TestPoint
- added TP501: VUSB, RD-Testpoints:TestPoint_Pad_D1.0mm, symbol Connector:TestPoint
- added TP601, TP602, TP603, TP604: TestPoint_PMK_Probe, RD-Testpoints:TestPoint_THTPad_PMK, symbol Ryan-Dynamics:TestPoint_PMK_Probe
- added U401: TPS7A2030PDBVR, Package_TO_SOT_SMD:SOT-23-5, symbol TPS7A2030PDBVR:TPS7A2030PDBVR
- added U501: STM32G441KBT6, Package_QFP:LQFP-32_7x7mm_P0.8mm, symbol MCU_ST_STM32G4:STM32G441KBTx
- added U502: USBLC6-2SC6, Package_TO_SOT_SMD:SOT-23-6, symbol Power_Protection:USBLC6-2SC6
- added U601, U602, U604, U605: TSV912AIDR, Package_SO:SOIC-8_3.9x4.9mm_P1.27mm, symbol Amplifier_Operational:TSV912IDT
- added U603, U701, U702: LM358LVIDR, Package_SO:SOIC-8_3.9x4.9mm_P1.27mm, symbol Amplifier_Operational:LM358
- added Y501: ATS08A-E, Crystal:Crystal_HC49-4H_Vertical, symbol Device:Crystal
Connections:
- new net: D502.2 (A), R502.1
- new net: R508.1, U501.31 (PB8)
- new net: J501.12 (~{RST}), R505.1
- new net: R623.1, R624.2, U601.5 (+)
- new net: J501.4 (JTMS/SWDIO), R504.1
- new net: J501.6 (JCLK/SWCLK), R503.1
- new net: J501.8 (JTDO/SWO), R506.1
- new net: D501.2 (A), R501.1
- new net +3V0: C405.2, C504.2, C506.2, C509.2, C512.2, C601.1, C602.1, C610.1, C614.1, C616.1, C701.1, C702.1, D601.1 (K), D603.1 (K), D605.1 (K), FB501.2, J501.3 (VCC), R623.2, R705.2, TP403.1, U401.5 (OUT), U501.1 (VDD), U501.17 (VDD), U502.5 (VBUS), U601.8 (V+), U602.8 (V+), U603.8 (V+), U604.8 (V+), U605.8 (V+), U701.8 (V+), U702.8 (V+)
- new net A+: U501.22 (PA12), U502.4 (I/O2)
- new net A-: U501.21 (PA11), U502.6 (I/O1)
- new net ADC_CE: R615.2, U501.12 (PA7)
- new net ADC_CO2: R619.2, U501.6 (PA1)
- new net ADC_ECG: R620.2, U501.5 (PA0)
- new net BTN: C501.2, SW501.2, U501.18 (PA8)
- new net CC1: J502.A5 (CC1), R509.2
- new net CC2: J502.B5 (CC2), R510.2
- new net CE_BUFF: R606.1, U603.1, U603.2 (-)
- new net CE_BUFF_IN: D603.2 (A), D604.1 (K), R602.2, U603.3 (+)
- new net CE_FILT: C608.1, R612.2, R615.1, TP602.1, U603.7
- new net CE_IN: J602.1 (In), R602.1
- new net CE_SK_MID: C608.2, R606.2, R609.1
- new net CE_SK_N: R611.2, R612.1, U603.6 (-)
- new net CE_SK_RC: C605.1, R609.2, U603.5 (+)
- new net CO2_BUFF: R607.1, U601.1, U601.2 (-)
- new net CO2_BUFF_IN: D605.2 (A), D606.1 (K), R603.2, U601.3 (+)
- new net CO2_FILT: C609.1, U602.1, U602.2 (-), U602.5 (+)
- new net CO2_GAIN_N: R613.2, R617.1, U602.6 (-)
- new net CO2_IN: J603.1 (In), R603.1
- new net CO2_OUT: R617.2, R619.1, TP603.1, U602.7
- new net CO2_SK_MID: C609.2, R607.2, R610.1
- new net CO2_SK_RC: C606.1, R610.2, U602.3 (+)
- new net D+: J502.A6 (D+), J502.B6 (D+), U502.3 (I/O2)
- new net D-: J502.A7 (D-), J502.B7 (D-), U502.1 (I/O1)
- new net DAC_SHAKER: R701.1, U501.9 (PA4)
- new net ECG_FILT: C607.1, R614.1, TP601.1, U604.6 (-), U604.7
- new net ECG_GAIN_N: R614.2, R616.2, R618.1, U605.2 (-)
- new net ECG_IN: J601.1 (In), R601.1
- new net ECG_LPF1: C603.1, R604.1, R605.1, U604.1
- new net ECG_LPF1_N: C603.2, D601.2 (A), D602.1 (K), R601.2, R604.2, U604.2 (-)
- new net ECG_OUT: R618.2, R620.1, R622.2, TP604.1, U605.1
- new net ECG_SK_MID: C607.2, R605.2, R608.1
- new net ECG_SK_RC: C604.1, R608.2, U604.5 (+)
- new net GATE_RPP: D401.2 (A), Q401.1, R401.1, R402.1
- new net GND: C401.2, C402.2, C403.2, C404.1, C405.1, C501.1, C502.1, C503.2, C504.1, C505.2, C506.1, C507.1, C508.2, C509.1, C510.1, C511.1, C512.1, C601.2, C602.2, C604.2, C605.2, C606.2, C610.2, C613.2, C614.2, C615.1, C616.2, C701.2, C702.2, C703.2, C705.2, C707.2, D501.1 (K), D502.1 (K), D503.2 (A2), D602.2 (A), D604.2 (A), D606.2 (A), H401.1, H402.1, H403.1, H404.1, J401.2, J402.1 (Pin_1), J501.5 (GND), J501.7 (GND), J502.A1 (GND), J502.A12 (GND), J502.B1 (GND), J502.B12 (GND), J502.S1 (SHIELD), J601.2 (Ext), J602.2 (Ext), J603.2 (Ext), R401.2, R508.2, R509.1, R510.1, R611.1, R613.1, R624.1, R706.1, SW501.1, TP404.1, TP601.2, TP602.2, TP603.2, TP604.2, U401.2 (GND), U501.14 (VSSA), U501.16 (VSS), U501.32 (VSS), U502.2 (GND), U601.4 (V-), U602.4 (V-), U603.4 (V-), U604.4 (V-), U605.4 (V-), U701.4 (V-), U702.4 (V-)
- new net LED_GRN: R501.2, U501.20 (PA10)
- new net LED_RED: R502.2, U501.19 (PA9)
- new net OSC_IN: C502.2, U501.2 (PF0), Y501.1
- new net OSC_OUT: R507.2, U501.3 (PF1)
- new net SERVO_N: C611.1, R621.1, U605.6 (-)
- new net SERVO_OUT: C611.2, R616.1, U605.7
- new net SERVO_P: C612.2, R622.1, U605.5 (+)
- new net SHAKER_N: J701.2 (Pin_2), R708.1, R709.2, U702.7
- new net SHAKER_P: J701.1 (Pin_1), R709.1, U702.1, U702.2 (-)
- new net SHK_FILT1: C704.1, R703.1, U701.1, U701.2 (-)
- new net SHK_FILT2: C706.1, R707.1, U701.6 (-), U701.7, U702.3 (+)
- new net SHK_N: R707.2, R708.2, U702.6 (-)
- new net SHK_SK1_MID: C704.2, R701.2, R702.1
- new net SHK_SK1_RC: C703.1, R702.2, U701.3 (+)
- new net SHK_SK2_MID: C706.2, R703.2, R704.1
- new net SHK_SK2_RC: C705.1, R704.2, U701.5 (+)
- new net SWCLK: R503.2, U501.24 (PA14)
- new net SWDIO: R504.2, U501.23 (PA13)
- new net SWO: R506.2, U501.26 (PB3)
- new net VBATT: C402.1, C403.1, D401.1 (K), JP401.1 (A), Q401.3, R402.2, TP402.1
- new net VBATT_FUSED: F401.2, Q401.2
- new net VBATT_RAW: F401.1, J401.1, J402.2 (Pin_2), TP401.1
- new net VBUS: F501.1, J502.A4 (VBUS), J502.A9 (VBUS), J502.B4 (VBUS), J502.B9 (VBUS)
- new net VDDA: C510.2, C511.2, FB501.1, U501.15 (VDDA)
- new net VIN_SEL: C401.1, C404.2, JP401.2 (C), U401.1 (IN), U401.3 (EN)
- new net VREF_ECG: C612.1, C613.1, C615.2, R621.2, U601.6 (-), U601.7, U604.3 (+), U605.3 (+)
- new net VREF_SHK: C707.1, R705.1, R706.2, U702.5 (+)
- new net VUSB: C505.1, C508.1, D503.1 (A1), F501.2, JP401.3 (B), TP501.1
- new net XTAL: C503.1, R507.1, Y501.2
- new net ~{RST}: C507.2, R505.2, U501.4 (PG10)
- no-connect marks 0 -> 18
Other:
- removed sheet ANALOGUE INPUTS
- removed sheet ANALOGUE OUTPUTS
- removed sheet DIGITAL AND HMI
- removed sheet POWER
- note added: "0.54V"
- note added: "0.59V"
- note added: "0.60V"
- note added: "0.61V"
- note added: "0.65V"
- note added: "1.0V"
- note added: "2ND ORDER NON-UNITY SK BWORTH LPF"
- note added: "2ND ORDER SK BWORTH LPF"
- note added: "3RD ORDER SK BWORTH LPF"
- note added: "4TH ORDER UNITY SK BWORTH RECONSTRUCTION FILTER"
- note added: "DC SERVO"
- note added: "DIFFERENTIAL OUTPUT DRIVER"
- note added: "GAIN STAGE"
- note added: "IC POWER AND DECOUPLING"
- note added: "MARKINGS"
- note added: "MOUNTING"
- note removed: "Page 4"
- note removed: "Page 5"
- note removed: "Page 6"
- note removed: "Page 7"
- title: ARCHITECTURE -> CIRCUIT
